Commit message: Harden companion robot operating modes

File: src/my_robot_package/urdf/my_robot.urdf (robot description, URDF)
Before this commit: robot my_robot, 7 links, 6 joints
Links:
- added link oakd_link
- added link oakd_rgb_camera_optical_frame
Joints:
- added joint oakd_joint: type fixed, parent base_link, child oakd_link, origin xyz=0.07 0 0.14 rpy=0 0 0
- added joint oakd_rgb_optical_joint: type fixed, parent oakd_link, child oakd_rgb_camera_optical_frame, origin xyz=0 0 0 rpy=-1.5708 0 -1.5708
